File: WiFi-Gate-Controller.kicad_pcb (KiCad board)
At the start: 2 copper layers, 66 x 51.5 mm, 91 parts, among them J1 Screw_Terminal_01x10, J2 USB_B_Micro, J3 Cortex Debug, SW1 Reset, U1 BTS3800SL, U10 SAMD21G18-M, U11 74LVC2G14, U12 74LVC2G14, U2 LMZ21700, U3 BTS3800SL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

Commit message: Arduino library updates.
Cleanup BOM.
Support KiBom.
Parts:
- C1, C2, C3, C4: value 1nF -> 1000pF
- C7: value 3.3nF -> 3300pF
- L1, L2, L3, L5: value 1k@1MHz -> 1k@100MHz
- L4: value 470@1MHz -> 470@100MHz
- R14: value 39 -> 39R
- R17: value 330 -> 330R
Connections:
- net VCC renamed +3V3
