File: WiFi-Gate-Controller.sch (KiCad schematic (older format))
At the start: 86 parts, among them J1 Screw_Terminal_01x10, J2 USB_B_Micro, J3 Cortex Debug, SW1 Reset, U1 BTS3800SL, U10 SAMD21G18-M, U11 74LVC2G14, U12 74LVC2G14, U2 LMZ21700, U3 BTS3800SL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

Commit message: Update to KiCad 5.1 libraries.
Also updated custom libraries.
Parts:
- C1, C10, C11, C12, C13, C14, C15, C16, C17, C18, C2, C20, C3, C4, C7, C9: footprint Capacitors_SMD:C_0603 -> Capacitor_SMD:C_0603_1608Metric; symbol device:C_Small -> Device:C_Small
- C19, C6, C8: footprint Capacitors_SMD:C_0805 -> Capacitor_SMD:C_0805_2012Metric; symbol device:C_Small -> Device:C_Small
- C5: footprint Capacitors_SMD:CP_Elec_8x10 -> Capacitor_SMD:CP_Elec_8x10; symbol device:CP_Small -> Device:CP_Small
- D1, D4, D5, D6: footprint TO_SOT_Packages_SMD:SOT-23 -> Package_TO_SOT_SMD:SOT-23; symbol ESD_Protection:NUP2105L -> Power_Protection-ML:NUP2105L
- D10: footprint TO_SOT_Packages_SMD:SOT-143 -> Package_TO_SOT_SMD:SOT-143; symbol ESD_Protection:PRTR5V0U2X -> Power_Protection-ML:PRTR5V0U2X
- D11, D12, D13, D15: footprint LEDs:LED_0603 -> LED_SMD:LED_0603_1608Metric; symbol device:LED_ALT -> Device:LED_ALT
- D14, D16, D17, D8, D9: footprint TO_SOT_Packages_SMD:SOT-23 -> Package_TO_SOT_SMD:SOT-23; symbol ti-ml:TPD2E2U06-Q1 -> Power_Protection-ML:TPD2E2U06
- D2, D3: footprint Diodes_SMD:D_PowerDI-123 -> Diode_SMD:D_PowerDI-123; symbol device:D_Schottky_ALT -> Device:D_Schottky_ALT
- D7: footprint Diodes_SMD:D_SMC -> Diode_SMD:D_SMC; symbol device:D_TVS_ALT -> Device:D_TVS_ALT
- J2: footprint Connectors_USB:USB_Micro-B_Wuerth-614105150721_Vertical_CircularHoles -> Connector_USB:USB_Micro-B_Wuerth_614105150721_Vertical_CircularHoles
- J3: footprint Pin_Headers:Pin_Header_Straight_2x05_Pitch1.27mm_SMD -> Connector_PinHeader_1.27mm:PinHeader_2x05_P1.27mm_Vertical_SMD; symbol Connector:Conn_02x05_Odd_Even -> Connector_Generic:Conn_02x05_Odd_Even
- JP1: footprint Pin_Headers:Pin_Header_Straight_2x01_Pitch2.54mm -> Connector_PinHeader_2.54mm:PinHeader_2x01_P2.54mm_Vertical; symbol device:Jumper_NC_Small -> Device:Jumper_NC_Small
- L1, L2, L3, L5: footprint Inductors_SMD:L_1206 -> Inductor_SMD:L_1206_3216Metric; symbol device:Ferrite_Bead -> Device:Ferrite_Bead
- L4: footprint Inductors_SMD:L_0603 -> Inductor_SMD:L_0603_1608Metric; symbol device:Ferrite_Bead -> Device:Ferrite_Bead
- R1, R12, R14, R16, R17, R2, R3, R7, R8, R9: footprint Resistors_SMD:R_0603 -> Resistor_SMD:R_0603_1608Metric; symbol device:R -> Device:R
- R10, R11, R13, R15, R18, R20, R21, R22, R23, R24, R25, R26, R27, R4, R5, R6: footprint Resistors_SMD:R_1206 -> Resistor_SMD:R_1206_3216Metric; symbol device:R -> Device:R
- SW1: footprint Buttons_Switches_SMD:SW_SPST_B3U-1000P -> Button_Switch_SMD:SW_SPST_B3U-1000P
- U1, U3, U4, U6: footprint infineon-ml:SCT595 -> Package_TO_SOT_SMD-ML:Infineon_PG-SCT595-5-1; symbol infineon-ml:BTS3800SL -> Power_Management-ML:BTS3800SL
- U10: footprint Housings_DFN_QFN:QFN-48-1EP_7x7mm_Pitch0.5mm -> Package_DFN_QFN:QFN-48-1EP_7x7mm_P0.5mm_EP5.15x5.15mm; symbol atmel-ml:SAMD21G18-M -> MCU_Microchip_SAMD-ML:SAMD21G18-M
- U11, U12, U7, U9: footprint TO_SOT_Packages_SMD:SOT-23-6 -> Package_TO_SOT_SMD:SOT-23-6; symbol Logic_74xgxx:74LVC2G14 -> 74xGxx:74LVC2G14
- U2: footprint ti-ml:SIL0008E -> Converter_DCDC-ML:Converter_DCDC_Texas-SIL0008E; symbol ti-ml:LMZ21700 -> Converter_DCDC-ML:LMZ21700
- U5: footprint Housings_SSOP:MSOP-8_3x3mm_Pitch0.65mm -> Package_SO:MSOP-8_3x3mm_P0.65mm; symbol sensors:DS18B20U -> Sensor_Temperature:DS18B20U
- U8: footprint atmel-ml:ATWINC1500-MR210XB -> RF_Module-ML:Microchip_ATWINC1500-MR210UB; symbol atmel-ml:ATWINC1500-MR210UB -> RF_WiFi-ML:ATWINC1500-MR210UB
- Y1: footprint abracon-ml:ABS07 -> Crystal-ML:Crystal_SMD_Abracon_ABS07-2Pin_3.2x1.5mm; symbol device:Crystal -> Device:Crystal
Other:
- note added: "The SAMD21G18 does not have extra filtering on the analog power supply so analog measurements may not be ideal."
- note removed: "The SAMD21G18 does not have extra filtering on the analog power supply so analog measurements may be ideal."

Commit message: Arduino library updates.
Cleanup BOM.
Support KiBom.
Parts:
- C1, C2, C3, C4: value 1nF -> 1000pF; Description (none) -> CAP, 0603, 1000pF, 10%, X7R, 10V
- C10, C11, C12, C13, C15, C18: Description (none) -> CAP, 0603, 0.1uF, 20%, X7R, 10V
- C14, C20: Description (none) -> CAP, 0603, 1uF, 10%, X7R, 10V
- C16, C17: Description (none) -> CAP, 0603, 15pF, 5%, C0G, 50V
- C19, C6: Description (none) -> CAP, 0805, 22uf, 20%, X5R, 25V
- C5: Description (none) -> CAP, SMD 8X10, 20%, EC, 35V
- C7: value 3.3nF -> 3300pF; Description (none) -> CAP, 0603, 3300pF, 5%, X7R, 10V
- C8: Description (none) -> CAP, 0805, 22uf, 20%, X5R, 25V; Vendor Part Number 810-C2012X5R1A226M-3 -> 963-TMK212BBJ226MGTT
- C9: Description (none) -> CAP, 0603, 0.1uF, 20%, X7R, 10V; Vendor Part Number 963-TMK212BBJ226MGTT -> 77-VJ0603Y104JXQPBC
- D1, D4, D5, D6: Description (none) -> TVS, SOT23, ESD Protection, CAN, 24V
- D10: Description (none) -> TVS, SOT23, ESD Protection, USB
- D11: Description (none) -> LED, 0603, Red
- D12: Description (none) -> LED, 0603, Yellow
- D13: Description (none) -> LED, 0603, Green
- D14, D16, D17, D8, D9: Description (none) -> TVS, SOT23, ESD TVS Protection, Dual
- D15: Description (none) -> LED, 0603, Orange
- D2, D3: Description (none) -> DIO, PowerDI123, Schottky Rectifier, 30V, 1A
- D7: Description (none) -> TVS, SMC, Transil, 1500W, 33V
- J1: Description (none) -> CON, THT, Terminal Block, Pluggable, 3.5mm, 10 Pos
- J2: Description (none) -> CON, THT, Micro USB 2.0 Type AB, Vertical
- J3: Description (none) -> CON, SMD, 1.27mm Header, Dual Row, Vertical, 10 Pos
- JP1: Description (none) -> CON, THT, 2.54mm Header, Single Row, Vertical, 2 Pos
- L1, L2, L3, L5: value 1k@1MHz -> 1k@100MHz; Description (none) -> BEAD, 1206, 1k@100MHz, 2A
- L4: value 470@1MHz -> 470@100MHz; Description (none) -> BEAD, 0603, 470R@100MHz, 1A
- R1: Description (none) -> RES, 0603, 1.21M, 1%, T100
- R10, R11, R13, R15, R18, R20, R21, R22, R23, R24, R25, R26, R27, R4, R5, R6: Description (none) -> RES, 1206, 100k, 5%, T200
- R12, R7, R8, R9: Description (none) -> RES, 0603, 1k, 1%, T100
- R14: value 39 -> 39R; Description (none) -> RES, 0603, 39R, 1%, T100
- R16: Description (none) -> RES, 0603, 10k, 1%, T100
- R17: value 330 -> 330R; Description (none) -> RES, 0603, 330R, 1%, T100
- R2: Description (none) -> RES, 0603, 383k, 1%, T100
- R3: Description (none) -> RES, 0603, 4.7k, 1%, T100
- SW1: Description (none) -> SW, SMD, Push Button
- U1, U3, U4, U6: Description (none) -> IC, SCT595, Smart Low Side Switch, 41V, 350mA
- U10: Description (none) -> IC, QFN44, MCU, ARM, 256kB Flash, 32kB SRAM, 48MHz
- U11, U12, U7, U9: Description (none) -> IC, SOT23-6, Dual inverting Schmitt trigger
- U2: Description (none) -> MODULE, SMD, Simple Switcher, 17V, 650mA
- U5: Description (none) -> IC, MSOP8, 1-Wire Temperature Sensor
- U8: Description (none) -> MODULE, SMD, WiFi, u.FL connector
- Y1: Description (none) -> XTL, SMD, 32.768kHz
Connections:
- net VCC renamed +3V3
